Commit message: feat(stage3): Intel RealSense D435i RGB-D camera integration
URDF / Kinematic Model:
  _properties.xacro  — Section 6: D435i physical constants (mass=72g,
    body=90x25x25mm, computed inertia tensor, D435i datasheet optical
    params: color FOV=69.4deg, depth FOV=86.0deg, clip 0.105-10.0m)
  _sensors.xacro     — Full D435i TF chain (REP-103 + RealSense SDK):
    camera_mount_link -> camera_link -> camera_color_frame
    -> camera_color_optical_frame (optical rpy=-pi/2,0,-pi/2)
    camera_link -> camera_depth_frame -> camera_depth_optical_frame
  _gazebo.xacro      — Gazebo Harmonic rgbd_camera sensor plugin:
    type=rgbd_camera, topic=camera/image_raw, update_rate=30Hz,
    gz_frame_id=camera_color_optical_frame, ideal noise mode (default)

Configuration:
  camera.yaml        — All D435i parameters: resolution, FPS, FOV, clip,
    dual noise modes (ideal/realistic), topic names, TF frame IDs,
    diagnostics thresholds, benchmark settings
  gz_bridge.yaml     — Stage 3: 5 new camera bridges added:
    /camera/color/image_raw, /camera/color/camera_info,
    /camera/depth/image_rect_raw, /camera/depth/camera_info,
    /camera/depth/points

Nodes:
  camera_diagnostics_node.py — monitors RGB/Depth/PC FPS (rolling
    window), per-stream latency, dropped frames, CPU%, RAM.
    Publishes diagnostic_msgs/DiagnosticArray -> /camera/diagnostics

Launch:
  controllers.launch.py — camera_diagnostics_node at t=10s
    (after gz_bridge stabilises), loads camera.yaml params

Validation:
  validate_camera.sh  — 9 automated test groups: topics, CameraInfo,
    RGB/Depth/PC FPS, TF tree completeness, frame_ids, stale topics
  benchmark_camera.py — timed benchmark (configurable duration/warmup),
    CSV output, pass/fail summary vs acceptance criteria

Build validation:
  13 links (was 8), 12 joints (was 7)
  All 11 camera links+joints: PASS
  colcon build: 4 packages, 0 errors, 1.15s

File: Simulation/vacuum_ws/src/vacuum_description/urdf/_gazebo.xacro (robot description, xacro)
@@ -55,4 +55,9 @@
     <selfCollide>false</selfCollide>
   </gazebo>
+  <!-- Stage 3: camera_link — D435i body -->
+  <gazebo reference="camera_link">
+    <material>Gazebo/DarkGrey</material>
+    <selfCollide>false</selfCollide>
+  </gazebo>
   <gazebo reference="arm_mount_link">
     <material>Gazebo/Yellow</material>
@@ -64,5 +69,5 @@
   </gazebo>
   <!-- ═══════════════════════════════════════════════════════
-       2. gz_ros2_control PLUGIN (Stage 2 — Gazebo Harmonic)
+       3. gz_ros2_control PLUGIN (Stage 2 — unchanged)
        ═══════════════════════════════════════════════════════ -->
   <!--
@@ -72,8 +77,8 @@
     _ros2_control.xacro.
     ros2_control then runs:
-      • diff_drive_controller  → publishes /odom, /tf, subscribes /cmd_vel
-      • joint_state_broadcaster → publishes /joint_states
+      - diff_drive_controller  -> publishes /odom, /tf, subscribes /cmd_vel
+      - joint_state_broadcaster -> publishes /joint_states
     All topics are native ROS2 — no ros_gz_bridge needed for them.
-    Only /clock still requires bridging.
+    Only /clock and camera topics still require bridging.
     Hardware transition (Jetson):
       Replace 'gz_ros2_control/GazeboSimSystem' in _ros2_control.xacro only.
@@ -92,3 +97,89 @@
     </plugin>
   </gazebo>
+  <!-- ═══════════════════════════════════════════════════════
+       4. INTEL REALSENSE D435i — RGB-D CAMERA SENSOR (Stage 3)
+       ═══════════════════════════════════════════════════════ -->
+  <!--
+    Sensor type: rgbd_camera (Gazebo Harmonic gz-sensors 8.x)
+    Attached to: camera_link (physical D435i body centre)
+    Topic layout generated by rgbd_camera sensor:
+      /camera/image_raw               -> colour image  (gz.msgs.Image)
+      /camera/image_raw/depth_image   -> depth image   (gz.msgs.Image)
+      /camera/image_raw/points        -> point cloud   (gz.msgs.PointCloudPacked)
+      /camera/image_raw/camera_info   -> colour info   (gz.msgs.CameraInfo)
+    These are bridged to standard ROS topics in gz_bridge.yaml:
+      /camera/color/image_raw
+      /camera/depth/image_rect_raw
+      /camera/depth/points
+      /camera/color/camera_info
+      /camera/depth/camera_info
+    gz_frame_id sets the frame_id in published image headers.
+    The TF tree (built from _sensors.xacro) makes the transforms available.
+    Noise modes (switch via camera.yaml noise_mode param — no code change):
+      ideal:     no noise (default for initial validation)
+      realistic: Gaussian depth + colour noise (for EKF/SLAM testing)
+    Prerequisites:
+      gz-sensors-rgbd-camera is included with Gazebo Harmonic.
+      No extra apt packages needed beyond ros-jazzy-ros-gz-bridge.
+    Sim-to-real:
+      Remove this gazebo block.
+      Launch realsense2_camera driver instead.
+      Downstream software unchanged.
+  -->
+  <gazebo reference="camera_link">
+    <sensor name="d435i" type="rgbd_camera">
+      <camera>
+        <!-- ── Colour channel ── -->
+        <horizontal_fov>${d435i_color_hfov}</horizontal_fov>
+        <image>
+          <width>${d435i_color_width}</width>
+          <height>${d435i_color_height}</height>
+          <format>R8G8B8</format>
+        </image>
+        <clip>
+          <near>${d435i_near_clip}</near>
+          <far>${d435i_far_clip}</far>
+        </clip>
+        <!-- ── Depth channel ── -->
+        <depth_camera>
+          <output>depths</output>
+          <clip>
+            <near>${d435i_near_clip}</near>
+            <far>${d435i_far_clip}</far>
+          </clip>
+        </depth_camera>
+        <!--
+          Ideal noise mode (default):
+            mean=0, stddev=0 — perfect depth, perfect colour.
+          Realistic noise mode:
+            Set mean=0, stddev=0.005 for ~5mm depth error at 1m.
+            Controlled via camera.yaml at runtime.
+        -->
+        <noise>
+          <type>gaussian</type>
+          <mean>0.0</mean>
+          <stddev>0.0</stddev>
+        </noise>
+      </camera>
+      <!-- Update at 30 Hz — matches D435i hardware default -->
+      <always_on>1</always_on>
+      <update_rate>${d435i_color_fps}</update_rate>
+      <visualize>false</visualize>
+      <!--
+        Gazebo topic root.
+        rgbd_camera generates sub-topics:
+          /camera/image_raw              -> colour image
+          /camera/image_raw/depth_image  -> depth image
+          /camera/image_raw/points       -> PointCloud2
+          /camera/image_raw/camera_info  -> CameraInfo
+      -->
+      <topic>camera/image_raw</topic>
+      <!--
+        gz_frame_id: sets frame_id in published ROS messages.
+        Using camera_color_optical_frame so image consumers get
+        the correct optical frame immediately.
+      -->
+      <gz_frame_id>camera_color_optical_frame</gz_frame_id>
+    </sensor>
+  </gazebo>
 </robot>

File: Simulation/vacuum_ws/src/vacuum_description/urdf/_properties.xacro (robot description, xacro)
@@ -118,3 +118,52 @@
   <xacro:property name="vacuum_mount_z"
     value="${-(chassis_height/2 + vacuum_mount_height/2)}"/>  <!-- = -0.055 -->
+  <!-- ==========================================================
+       6. INTEL REALSENSE D435i  (Stage 3)
+          All values sourced from Intel D435i datasheet v0.9.
+       ========================================================== -->
+  <!-- D435i body: 90mm W x 25mm H x 25mm D, 72g -->
+  <xacro:property name="d435i_body_x" value="0.025"/>  <!-- depth into scene -->
+  <xacro:property name="d435i_body_y" value="0.090"/>  <!-- width -->
+  <xacro:property name="d435i_body_z" value="0.025"/>  <!-- height -->
+  <xacro:property name="d435i_mass"   value="0.072"/>  <!-- kg -->
+  <!--
+    camera_link inertia (box, m=0.072kg, x=0.025m, y=0.090m, z=0.025m):
+      Ixx=(1/12)*m*(y^2+z^2) = (1/12)*0.072*(0.0081+0.000625) = 5.24e-5
+      Iyy=(1/12)*m*(x^2+z^2) = (1/12)*0.072*(0.000625+0.000625) = 7.5e-6
+      Izz=(1/12)*m*(x^2+y^2) = (1/12)*0.072*(0.000625+0.0081)   = 5.24e-5
+  -->
+  <xacro:property name="d435i_ixx" value="0.0000524"/>
+  <xacro:property name="d435i_iyy" value="0.0000075"/>
+  <xacro:property name="d435i_izz" value="0.0000524"/>
+  <!-- camera_link offset from camera_mount_link (sits on top) -->
+  <xacro:property name="camera_link_x" value="0.0"/>
+  <xacro:property name="camera_link_y" value="0.0"/>
+  <xacro:property name="camera_link_z"
+    value="${camera_mount_height/2 + d435i_body_z/2}"/>  <!-- = 0.025 -->
+  <!-- colour module: +11.5mm right on real hw; co-located in sim -->
+  <xacro:property name="camera_color_x" value="0.0"/>
+  <xacro:property name="camera_color_y" value="0.0"/>
+  <xacro:property name="camera_color_z" value="0.0"/>
+  <!-- depth module: at body centre on real hw -->
+  <xacro:property name="camera_depth_x" value="0.0"/>
+  <xacro:property name="camera_depth_y" value="0.0"/>
+  <xacro:property name="camera_depth_z" value="0.0"/>
+  <!--
+    Optical frame rotation: robot convention (x-fwd) to optical (z-fwd,x-right,y-down)
+    rpy = "-pi/2  0  -pi/2"
+  -->
+  <xacro:property name="optical_roll"  value="-1.5707963"/>
+  <xacro:property name="optical_pitch" value="0.0"/>
+  <xacro:property name="optical_yaw"   value="-1.5707963"/>
+  <!-- D435i Gazebo sensor parameters (baked at Xacro expansion; tune via camera.yaml) -->
+  <xacro:property name="d435i_color_width"  value="640"/>
+  <xacro:property name="d435i_color_height" value="480"/>
+  <xacro:property name="d435i_color_fps"    value="30"/>
+  <xacro:property name="d435i_color_hfov"   value="1.2112"/>  <!-- 69.4 deg -->
+  <xacro:property name="d435i_depth_width"  value="640"/>
+  <xacro:property name="d435i_depth_height" value="480"/>
+  <xacro:property name="d435i_depth_fps"    value="30"/>
+  <xacro:property name="d435i_depth_hfov"   value="1.5010"/>  <!-- 86.0 deg -->
+  <xacro:property name="d435i_near_clip"    value="0.105"/>  <!-- m -->
+  <xacro:property name="d435i_far_clip"     value="10.0"/>   <!-- m -->
 </robot>

File: Simulation/vacuum_ws/src/vacuum_description/urdf/_sensors.xacro (robot description, xacro)
@@ -1,18 +1,28 @@
 <?xml version="1.0"?>
 <!--
-  _sensors.xacro
-  ──────────────
-  Stage 1: Mounting point placeholders only — no sensor plugins yet.
-  Plugins (D435i RGB-D + IMU) will be added in Stage 3 (Sensors).
-  Links created:
-    camera_mount_link  — D435i camera position reference
-    arm_mount_link     — Robotic arm base attachment point
-    vacuum_mount_link  — Vacuum module attachment point
-  All joints are fixed (rigid mounts).
-  All links have minimal but non-zero mass for physical correctness.
+  _sensors.xacro  (Stage 3 — Intel RealSense D435i Integration)
+  ──────────────────────────────────────────────────────────────
+  Replaces the Stage 1/2 placeholder with a complete camera model.
+  TF chain produced (follows Intel RealSense SDK + REP-103):
+    base_link
+      └── camera_mount_link     (Stage 1 placeholder, physical chassis bracket)
+            └── camera_link     (D435i body geometric centre)
+                  ├── camera_color_frame          (colour sensor plane)
+                  │     └── camera_color_optical_frame   (ROS optical convention)
+                  └── camera_depth_frame          (depth sensor plane)
+                        └── camera_depth_optical_frame   (ROS optical convention)
+  Optical convention:
+    Standard frames (camera_*_frame):  x-forward, y-left, z-up
+    Optical frames (camera_*_optical): x-right, y-down, z-into-scene
+    Transform:  rpy = "-pi/2  0  -pi/2"
+  All numeric values are defined in _properties.xacro (Section 6).
+  Gazebo plugin (rgbd_camera sensor) lives in _gazebo.xacro.
+  Sim-to-real transfer note:
+    In hardware mode replace the Gazebo sensor with:
+      ros2 launch realsense2_camera rs_launch.py
+    No URDF changes needed — only the sensor plugin source changes.
 -->
 <robot xmlns:xacro="http://www.ros.org/wiki/xacro">
-  <!-- ── D435i Camera Mount ─────────────────────────────────────── -->
-  <!-- Front-top of chassis. The D435i will be attached here in Stage 3. -->
+  <!-- ── camera_mount_link (Stage 1 placeholder kept unchanged) ─── -->
   <xacro:mount_placeholder
     name="camera_mount"
@@ -26,6 +36,90 @@
     mass="${camera_mount_mass}"
     mat="dark_grey"/>
-  <!-- ── Robotic Arm Mount ──────────────────────────────────────── -->
-  <!-- Rear-top of chassis. MoveIt2 arm will be attached here in Stage 6. -->
+  <!-- ═══════════════════════════════════════════════════════
+       camera_link — physical body of the D435i
+       ═══════════════════════════════════════════════════════ -->
+  <!--
+    Sits on top of camera_mount_link.
+    z-offset = mount_height/2 + d435i_body_z/2  (see _properties.xacro).
+    This link represents the geometric centre of the D435i enclosure.
+  -->
+  <joint name="camera_joint" type="fixed">
+    <parent link="camera_mount_link"/>
+    <child  link="camera_link"/>
+    <origin xyz="${camera_link_x} ${camera_link_y} ${camera_link_z}"
+            rpy="0 0 0"/>
+  </joint>
+  <link name="camera_link">
+    <visual>
+      <origin xyz="0 0 0" rpy="0 0 0"/>
+      <geometry>
+        <box size="${d435i_body_x} ${d435i_body_y} ${d435i_body_z}"/>
+      </geometry>
+      <material name="dark_grey"/>
+    </visual>
+    <collision>
+      <origin xyz="0 0 0" rpy="0 0 0"/>
+      <geometry>
+        <box size="${d435i_body_x} ${d435i_body_y} ${d435i_body_z}"/>
+      </geometry>
+    </collision>
+    <inertial>
+      <origin xyz="0 0 0" rpy="0 0 0"/>
+      <mass value="${d435i_mass}"/>
+      <inertia
+        ixx="${d435i_ixx}" ixy="0" ixz="0"
+        iyy="${d435i_iyy}" iyz="0"
+        izz="${d435i_izz}"/>
+    </inertial>
+  </link>
+  <!-- ═══════════════════════════════════════════════════════
+       camera_color_frame  (colour sensor, robot convention)
+       camera_color_optical_frame  (colour sensor, optical convention)
+       ═══════════════════════════════════════════════════════ -->
+  <joint name="camera_color_joint" type="fixed">
+    <parent link="camera_link"/>
+    <child  link="camera_color_frame"/>
+    <origin xyz="${camera_color_x} ${camera_color_y} ${camera_color_z}"
+            rpy="0 0 0"/>
+  </joint>
+  <link name="camera_color_frame">
+    <!-- Massless optical frame — no visual/collision/inertial needed -->
+  </link>
+  <joint name="camera_color_optical_joint" type="fixed">
+    <parent link="camera_color_frame"/>
+    <child  link="camera_color_optical_frame"/>
+    <!--
+      Standard optical rotation: x-right, y-down, z-into-scene.
+      From robot convention: rpy = "-pi/2  0  -pi/2".
+    -->
+    <origin xyz="0 0 0"
+            rpy="${optical_roll} ${optical_pitch} ${optical_yaw}"/>
+  </joint>
+  <link name="camera_color_optical_frame">
+    <!-- Massless optical reference frame -->
+  </link>
+  <!-- ═══════════════════════════════════════════════════════
+       camera_depth_frame  (depth sensor, robot convention)
+       camera_depth_optical_frame  (depth sensor, optical convention)
+       ═══════════════════════════════════════════════════════ -->
+  <joint name="camera_depth_joint" type="fixed">
+    <parent link="camera_link"/>
+    <child  link="camera_depth_frame"/>
+    <origin xyz="${camera_depth_x} ${camera_depth_y} ${camera_depth_z}"
+            rpy="0 0 0"/>
+  </joint>
+  <link name="camera_depth_frame">
+    <!-- Massless optical frame -->
+  </link>
+  <joint name="camera_depth_optical_joint" type="fixed">
+    <parent link="camera_depth_frame"/>
+    <child  link="camera_depth_optical_frame"/>
+    <origin xyz="0 0 0"
+            rpy="${optical_roll} ${optical_pitch} ${optical_yaw}"/>
+  </joint>
+  <link name="camera_depth_optical_frame">
+    <!-- Massless optical reference frame -->
+  </link>
+  <!-- ── Arm and vacuum mounts (unchanged from Stage 1) ─────────── -->
   <xacro:mount_placeholder
     name="arm_mount"
@@ -39,6 +133,4 @@
     mass="${arm_mount_mass}"
     mat="yellow"/>
-  <!-- ── Vacuum Module Mount ────────────────────────────────────── -->
-  <!-- Front-bottom of chassis. Vacuum module will be attached in Stage 4. -->
   <xacro:mount_placeholder
     name="vacuum_mount"
