Commit message: feat(stage4): completed manual slam mapping and map export in apartment world

File: Simulation/vacuum_ws/src/vacuum_description/urdf/_macros.xacro (robot description, xacro)
@@ -108,5 +108,5 @@
       <parent link="${parent}"/>
       <child  link="${name}_link"/>
-      <origin xyz="0 ${y_reflect * wheel_joint_y} ${wheel_joint_z}"
+      <origin xyz="${wheel_joint_x} ${y_reflect * wheel_joint_y} ${wheel_joint_z}"
               rpy="0 0 0"/>
       <axis xyz="0 1 0"/>

File: Simulation/vacuum_ws/src/vacuum_description/urdf/_properties.xacro (robot description, xacro)
@@ -78,5 +78,7 @@
        z_wheel_in_base_link = 0.033 - 0.093 = -0.060 m
        y_wheel = ± wheel_separation/2 = ± 0.134 m
+       x_wheel = drive wheels shifted behind geometric centre = -0.080 m
   -->
+  <xacro:property name="wheel_joint_x"   value="-0.080"/>
   <xacro:property name="wheel_joint_z"   value="-0.060"/>
   <xacro:property name="wheel_joint_y"   value="0.134"/>  <!-- half separation -->
